Commit message: tutorial

File: test.urdf (robot description, URDF)
Before this commit: robot UNNAMED_0, 7 links, 6 joints
Links:
- removed link L6
- removed link L7
- link L3: geometry collision box size=0.1 0.1 1.8002205420447797; visual box size=0.1 0.1 1.8002205420447797
- link L4: geometry collision box size=0.1 0.1 5.156238357562613; visual box size=0.1 0.1 5.156238357562613
- link L5: geometry collision box size=0.1 0.1 2.8000146428188546; visual box size=0.1 0.1 2.8000146428188546
Joints:
- removed joint G2
- removed joint Gabs
- removed joint J1b1
- removed joint J1b2
- removed joint J1m
- removed joint J2m
- added joint EE: type revolute, parent L4, child EE, origin xyz=1e-15 0.0 5.156238357562613 rpy=0.0 -1.2624159275672684 0.0, axis 0 1 0, limit lower=-3.141592653589793 upper=3.141592653589793 effort=2 velocity=10
- added joint J0: type revolute, parent G, child L3, origin xyz=0.0 0.0 0.0 rpy=0.0 0.6482783194240893 0.0, axis 0 1 0, limit lower=-3.141592653589793 upper=3.141592653589793 effort=2 velocity=10
- added joint J1: type revolute, parent L3, child L4, origin xyz=-0.0 0.0 1.80022054204478 rpy=0.0 0.6141376081431793 0.0, axis 0 1 0, limit lower=-3.141592653589793 upper=3.141592653589793 effort=2 velocity=10
- added joint J3: type revolute, parent G, child L5, origin xyz=4.2 0.0 0.0 rpy=0.0 0.46636282353891545 0.0, axis 0 1 0, limit lower=-3.141592653589793 upper=3.141592653589793 effort=2 velocity=10
