Commit message: update examples and apps, remove olds

File: parametrized_builder_test.urdf (robot description, URDF)
Before this commit: robot Robot, 21 links, 20 joints
Links:
- link G: mass 6.171428571428573 -> 64.00000000000001
- link L3: geometry collision box size=0.04 0.04 0.22448683107033715; visual box size=0.04 0.04 0.22448683107033715
- link L4: mass 1.6987621821860732 -> 1.6987621821860728; geometry collision box size=0.03999999910593033 0.03999999910593033 0.22448683196440689; collision box size=0.03999999910593033 0.03999999910593033 0.5000617257613914
Joints:
- removed joint 4L_top_L7_Weld
- removed joint 4L_top_L7_revolute
- added joint 4L_top_L6_Weld: type fixed, parent L7, child 4L_top_L7Pseudo, origin xyz=5.551115123125783e-17 0.0 0.28867513459481287 rpy=3.141592653589793 -1.286412781872945 3.141592653589793
- added joint 4L_top_L6_revolute: type revolute, parent L6, child 4L_top_L6Pseudo, origin xyz=-5.551115123125783e-17 0.0 0.2644868310703372 rpy=0.0 0.0 0.0, axis 0 1 0, limit lower=-3.141592653589793 upper=3.141592653589793 effort=600.0 velocity=6.283185307179586
- joint 2L_ground_G_WeldActuator: origin xyz=-0.5 0.03975 0.0 rpy=-1.5707963267948966 0.022584157122803594 -3.141592653589793 -> xyz=-0.5 0.03975 0.0 rpy=-1.570796326794897 0.022584157122803594 3.1415926535897927
- joint 2L_ground_G_WeldUnit: origin xyz=-0.5 0.0 0.0 rpy=-1.5707963267948966 0.022584157122803594 -3.141592653589793 -> xyz=-0.5 0.0 0.0 rpy=-1.570796326794897 0.022584157122803594 3.1415926535897927
- joint 4LT2_j0: origin xyz=3.885780586188048e-16 0.0 0.2644868310703371 rpy=0.0 -0.7853981633974468 0.0 -> xyz=3.885780586188048e-16 0.0 0.26448683107033705 rpy=0.0 -0.7853981633974468 0.0
- joint 4LT2_j0_L3_WeldUnit: origin xyz=3.885780586188048e-16 0.0 0.2644868310703371 rpy=1.5707963267948966 -0.7853981633974467 0.0 -> xyz=3.885780586188048e-16 0.0 0.26448683107033705 rpy=1.5707963267948966 -0.7853981633974468 0.0
- joint 4LT2_j1: origin xyz=0.0 0.0 0.2644868310703372 rpy=0.0 -0.785398163397448 0.0 -> xyz=0.0 0.0 0.2644868310703372 rpy=0.0 -0.7853981633974483 0.0
- joint 4LT2_j1_L4_WeldUnit: origin xyz=0.0 0.0 0.2644868310703372 rpy=1.5707963267948961 -0.7853981633974481 1.1102230246251565e-16 -> xyz=0.0 0.0 0.2644868310703372 rpy=1.5707963267948961 -0.7853981633974481 -1.1102230246251565e-16
- joint 4LT2_j2: origin xyz=5.551115123125783e-17 0.0 0.2644868310703372 rpy=0.0 -0.7853981633974483 0.0 -> xyz=0.0 0.0 0.2644868310703372 rpy=0.0 -0.7853981633974483 0.0
- joint 4LT2_j2_L5_WeldUnit: origin xyz=5.551115123125783e-17 0.0 0.2644868310703372 rpy=1.5707963267948966 -0.7853981633974484 1.1102230246251565e-16 -> xyz=0.0 0.0 0.2644868310703372 rpy=1.5707963267948961 -0.7853981633974483 1.1102230246251565e-16
- joint Main_ee_L8_WeldUnit: origin xyz=5.551115123125783e-17 0.0 0.5773502691896257 rpy=-1.5707963267948966 0.5235987755982987 -3.141592653589793 -> xyz=5.551115123125783e-17 0.0 0.5773502691896257 rpy=-1.5707963267948966 0.5235987755982991 -3.141592653589793
- joint Main_ground_G_WeldActuator: origin xyz=0.0 0.050999999552965164 0.0 rpy=-1.5707963267948966 0.5235987755982987 -3.141592653589793 -> xyz=0.0 0.050999999552965164 0.0 rpy=-1.5707963267948966 0.5235987755982991 -3.141592653589793
- joint Main_ground_G_WeldUnit: origin xyz=0.0 0.0 0.0 rpy=-1.5707963267948966 0.5235987755982987 -3.141592653589793 -> xyz=0.0 0.0 0.0 rpy=-1.5707963267948966 0.5235987755982991 -3.141592653589793
- joint Main_knee: origin xyz=-2.7755575615628914e-17 0.0 0.5773502691896257 rpy=0.0 1.0471975511965974 0.0 -> xyz=-2.7755575615628914e-17 0.0 0.5773502691896257 rpy=0.0 1.0471975511965979 0.0
- joint Main_knee_L7_WeldUnit: origin xyz=-2.7755575615628914e-17 0.0 0.5773502691896257 rpy=1.5707963267948966 1.0471975511965979 0.0 -> xyz=-2.7755575615628914e-17 0.0 0.5773502691896257 rpy=1.5707963267948961 1.0471975511965979 -2.220446049250313e-16
