Commit message: ge

File: robots/5bar_linkage_iso6d/robot.urdf (robot description, URDF)
Before this commit: robot onshape, 10 links, 9 joints
Links:
- removed link effecteur
- removed link part_1
- added link bout_pied, mass 1e-9
- added link centre_hanche, mass 92.082931928983427383; collision mesh filename=package:///part_1.stl; visual mesh filename=package:///part_1.stl
Joints:
- removed joint effecteur_frame
- added joint bout_pied_frame: type fixed, parent part_4, child bout_pied, origin xyz=0.025000000000000022204 -0.18000000000000015987 -0.067499999999999976685 rpy=-3.141592653589793116 -1.5132630134575502908e-16 -1.570796326794896558, axis 0 0 0
- joint libre2: parent part_1 -> centre_hanche
- joint mot1: parent part_1 -> centre_hanche

File: robots/talos_like/robot.urdf (robot description, URDF)
Before this commit: robot onshape, 14 links, 13 joints
Links:
- link buste: mass 0.423073581028333479 -> 110.423073581028333479
